File: mac-vintage-hdmi/mac-vintage-hdmi.kicad_pcb (KiCad board)
At the start: 2 copper layers, 4.5 x 13.4 mm, 201 parts, among them J1 HDMI_A, J10 Conn_02x05_Odd_Even, J11 Conn_02x05_Odd_Even, J12 Conn_02x05_Odd_Even, J2 USB_C_Receptacle_USB2.0_16P, J3 BM03B-SRSS-TB, J4 BM03B-SRSS-TB, J5 39-28-1143, J8 Conn_02x05_Odd_Even, J9 Conn_02x05_Odd_Even, Q1 Si2342DS, Q10 BSS123LT1, Q2 BSS123LT1, Q3 BSS123LT1, Q4 BSS123LT1, Q5 BSS123LT1, Q6 BSS123LT1, Q7 BSS123LT1, Q8 BSS123LT1, Q9 BSS123LT1, SW1 434133025816, SW2 434133025816, SW3 434133025816, U1 ADV7611, U10 LM66100DCKR, U2 TXU0104PWR, U3 RP2354B, U4 NCP1117-3.3_SOT223, U5 NCP1117-3.3_SOT223, U6 NCP1117ST18T3G, U7 NCP115AMX120TCG, U8 ICE40UP5K-SG48I, U9 LM66100DCKR, Y1 ABM8-272-T3, Y2 ABM8-28.63636MHZ-B2-T

Commit message: more placement
Parts:
- R68: footprint Resistor_SMD:R_01005_0402Metric_Pad0.57x0.30mm_HandSolder -> Resistor_SMD:R_0805_2012Metric_Pad1.20x1.40mm_HandSolder
- moved Q4 256.2 mm to (-163.5, 21.9)
- moved Q3 256.0 mm to (-163.5, 18.5), turned to 180 degrees
- moved R22 247.2 mm to (-166.5, 19.5), turned to -90 degrees
- moved Q2 247.2 mm to (-159.0, 21.0)
- moved D10 244.5 mm to (-156.0, 19.5), turned to 90 degrees
- moved R20 239.1 mm to (-159.0, 18.0)
- moved C15 229.5 mm to (48.5, 124.3)
- moved C16 229.5 mm to (49.5, 124.3)
- moved C54 229.5 mm to (46.5, 124.3)
- moved C55 229.5 mm to (57.0, 131.3)
- moved C56 229.5 mm to (57.5, 129.3)
- moved C57 229.5 mm to (63.0, 120.8)
- moved C58 229.5 mm to (61.0, 121.3)
- moved C59 229.5 mm to (49.0, 120.3)
- moved C60 229.5 mm to (51.0, 120.8)
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Connections:
- R68 pad 1: Net-(U2-OE) -> +5V
- R68 pad 2: +5V -> Net-(U2-OE)
Other:
- board text added: "1V1"
- board text added: "3V3"
- board text added: "5V"
- board text added: "BOOT"
- board text added: "GPIO"
- board text added: "HPD"
- board text added: "RESET_L"
- board text added: "RUN"
- board text added: "USB"

Commit message: ready for design review
Parts:
- removed C15, C16, C56, C58, C60, C61, C63, C66: 100n, Capacitor_SMD:C_0402_1005Metric_Pad0.74x0.62mm_HandSolder
- removed C54, C55, C57, C59, C62, C64, C65: 4.7uF, Capacitor_SMD:C_0805_2012Metric_Pad1.18x1.45mm_HandSolder
- removed D13: MHPA1010RGBDT, mac-vintage-hdmi:LED_RGB_Meihua_MHPA1010RGBDT_1x1mm
- removed J11: Conn_02x05_Odd_Even, mac-vintage-hdmi:PinHeader_2x05_P2.54mm_Vertical_SMD
- removed L1: 3.3uH, Inductor_SMD:L_0805_2012Metric_Pad1.05x1.20mm_HandSolder
- removed Q7, Q8: BSS123LT1, mac-vintage-hdmi:SOT-23
- removed R16: 10k, Resistor_SMD:R_0805_2012Metric_Pad1.20x1.40mm_HandSolder
- removed R27: 100k, Resistor_SMD:R_0805_2012Metric_Pad1.20x1.40mm_HandSolder
- removed R28: 5.1k, Resistor_SMD:R_0805_2012Metric_Pad1.20x1.40mm_HandSolder
- removed R37: 100, Resistor_SMD:R_01005_0402Metric_Pad0.57x0.30mm_HandSolder
- removed R45, R46, R47, R48, R49, R50, R51, R52, R53, R54, R55, R57, R63: 0, Resistor_SMD:R_01005_0402Metric_Pad0.57x0.30mm_HandSolder
- removed SW3: 434133025816, mac-vintage-hdmi:SW_Push_1P1T_NO_Vertical_Wuerth_434133025816
- removed U7: NCP115AMX120TCG, Package_DFN_QFN:OnSemi_XDFN4-1EP_1.0x1.0mm_EP0.52x0.52mm
- removed U8: ICE40UP5K-SG48I, mac-vintage-hdmi:QFN-48-1EP_7x7mm_P0.5mm_EP5.3x5.3mm
- added C73: 0.1uF, Capacitor_SMD:C_0805_2012Metric_Pad1.18x1.45mm_HandSolder, F.Cu at (122.1, 5.35)
- added C74: 47uF, Capacitor_SMD:C_1210_3225Metric_Pad1.33x2.70mm_HandSolder, F.Cu at (119.1, 5.35)
- added C75: 0.1uF, Capacitor_SMD:C_0805_2012Metric_Pad1.18x1.45mm_HandSolder, F.Cu at (129.0, 40.7)
- added C76: 10uF, Capacitor_SMD:C_0805_2012Metric_Pad1.18x1.45mm_HandSolder, F.Cu at (127.8, 45.2)
- added C77: 47uF, Capacitor_SMD:C_1210_3225Metric_Pad1.33x2.70mm_HandSolder, F.Cu at (120.5, 49.1)
- added C78: 47nF, Capacitor_SMD:C_0805_2012Metric_Pad1.18x1.45mm_HandSolder, F.Cu at (116.5, 43.7)
- added C79: 10uF, Capacitor_SMD:C_0805_2012Metric_Pad1.18x1.45mm_HandSolder, F.Cu at (123.0, 35.0)
- added C80: 0.1uF, Capacitor_SMD:C_0805_2012Metric_Pad1.18x1.45mm_HandSolder, F.Cu at (134.4, 16.0)
- added C81: 470pF, Capacitor_SMD:C_0805_2012Metric_Pad1.18x1.45mm_HandSolder, F.Cu at (130.9, 13.0)
- added C82: 1nF, Capacitor_SMD:C_0805_2012Metric_Pad1.18x1.45mm_HandSolder, F.Cu at (128.4, 16.0)
- added C83: 0.1uF, Capacitor_SMD:C_0402_1005Metric_Pad0.74x0.62mm_HandSolder, F.Cu at (19.0, 21.5)
- added C84: 47uF, Capacitor_SMD:C_1210_3225Metric_Pad1.33x2.70mm_HandSolder, F.Cu at (125.0, 50.0)
- added C85: 0.1uF, Capacitor_SMD:C_0805_2012Metric_Pad1.18x1.45mm_HandSolder, F.Cu at (124.0, 47.2)
- added FB1: BLM18KG601SN1D, mac-vintage-hdmi:L_0603_1608Metric_Pad1.05x0.95mm_HandSolder, F.Cu at (34.4, 13.0)
- added FB2: BLM18KG601SN1D, mac-vintage-hdmi:L_0603_1608Metric_Pad1.05x0.95mm_HandSolder, F.Cu at (31.2, 37.2)
- added FB3: BLM18KG601SN1D, mac-vintage-hdmi:L_0603_1608Metric_Pad1.05x0.95mm_HandSolder, F.Cu at (26.2, 34.2)
- added J6: Conn_01x02, mac-vintage-hdmi:PinHeader_1x02_P2.54mm_Vertical_SMD_Pin1Left, F.Cu at (60.5, 48.0)
- added L2: AOTA-B201610S3R3-101-T, mac-vintage-hdmi:L_Abracon_AOTA-B201610S3R3-101-T_2.0x1.6mm, F.Cu at (83.8, 41.0)
- added R76: 0, Resistor_SMD:R_0805_2012Metric_Pad1.20x1.40mm_HandSolder, F.Cu at (117.0, 55.8)
- added R77: 0, Resistor_SMD:R_0402_1005Metric_Pad0.72x0.64mm_HandSolder, F.Cu at (104.5, 35.1)
- added R78: 0, Resistor_SMD:R_0402_1005Metric_Pad0.72x0.64mm_HandSolder, F.Cu at (105.0, 46.5)
- added R79: 5.1k, Resistor_SMD:R_0805_2012Metric_Pad1.20x1.40mm_HandSolder, F.Cu at (129.0, 43.1)
- added R80: 47, Resistor_SMD:R_0805_2012Metric_Pad1.20x1.40mm_HandSolder, F.Cu at (118.5, 43.7)
- added R81: 0, Resistor_SMD:R_0402_1005Metric_Pad0.72x0.64mm_HandSolder, F.Cu at (125.9, 15.0)
- added R82: 13k, Resistor_SMD:R_0805_2012Metric_Pad1.20x1.40mm_HandSolder, F.Cu at (126.0, 11.8)
- added R83: 8.2k, Resistor_SMD:R_0805_2012Metric_Pad1.20x1.40mm_HandSolder, F.Cu at (127.9, 11.8)
- added R84: 0, Resistor_SMD:R_0402_1005Metric_Pad0.72x0.64mm_HandSolder, F.Cu at (103.8, 46.5)
- added RV1: PTV09A, mac-vintage-hdmi:Potentiometer_Bourns_PTV09A_RearMount, F.Cu at (121.5, 32.3)
- added TP4: TestPoint, TestPoint:TestPoint_Pad_2.0x2.0mm, F.Cu at (35.0, 9.00)
- added TP5: TestPoint, TestPoint:TestPoint_Pad_2.0x2.0mm, F.Cu at (133.6, 6.10)
- added U11: LM386M-1, mac-vintage-hdmi:SOIC-8_3.9x4.9mm_P1.27mm, F.Cu at (122.6, 42.0)
- added U12: PT8211-S, mac-vintage-hdmi:SOIC-8_3.9x4.9mm_P1.27mm, F.Cu at (126.3, 5.25)
- added U13: TLV9061IDBVR, mac-vintage-hdmi:SOT-23-5, F.Cu at (131.6, 16.2)
- C35: value 0.1uF -> 100n; footprint Capacitor_SMD:C_0805_2012Metric_Pad1.18x1.45mm_HandSolder -> Capacitor_SMD:C_0402_1005Metric_Pad0.74x0.62mm_HandSolder
- C37, C39: footprint Capacitor_SMD:C_0805_2012Metric_Pad1.18x1.45mm_HandSolder -> Capacitor_SMD:C_0402_1005Metric_Pad0.74x0.62mm_HandSolder
- C52: value 4.7uF -> 100n; footprint Capacitor_SMD:C_0805_2012Metric_Pad1.18x1.45mm_HandSolder -> Capacitor_SMD:C_0402_1005Metric_Pad0.74x0.62mm_HandSolder
- C53: value 4.7uF -> 10uF
- D12: value LED -> MA3X704A; footprint LED_SMD:LED_0805_2012Metric_Pad1.15x1.40mm_HandSolder -> mac-vintage-hdmi:SC-59
- J2: value USB_C_Receptacle_USB2.0_16P -> TYPE-C-31-M-12; footprint Connector_USB:USB_C_Receptacle_Amphenol_12401948E412A -> mac-vintage-hdmi:USB_C_Receptacle_HRO_TYPE-C-31-M-12
- R26: value 100k -> 27k
- R30, R32, R34, R36, R38, R39, R40, R41, R42, R43, R44, R56: value 0 -> 33; footprint Resistor_SMD:R_01005_0402Metric_Pad0.57x0.30mm_HandSolder -> Resistor_SMD:R_0402_1005Metric_Pad0.72x0.64mm_HandSolder
- R31: value 0 -> 2.7k
- R58, R59, R60, R61, R62, R64, R69: footprint Resistor_SMD:R_01005_0402Metric_Pad0.57x0.30mm_HandSolder -> Resistor_SMD:R_0402_1005Metric_Pad0.72x0.64mm_HandSolder
- R75: value 0 -> 1k
- U6: footprint mac-vintage-hdmi:SOT-223 -> mac-vintage-hdmi:SOT-223-3_TabPin2
- moved C35 220.2 mm to (80.5, 33.2), turned to 180 degrees
- moved C29 181.7 mm to (41.9, 24.8), turned to 90 degrees
- moved SW2 179.6 mm to (107.8, 5.50), turned to 180 degrees
- moved C20 179.0 mm to (34.4, 14.9)
- moved C47 178.7 mm to (44.4, 45.0), turned to -90 degrees
- moved C31 178.0 mm to (38.3, 15.0)
- moved Q9 177.3 mm to (102.1, 3.48), turned to 180 degrees
- moved C45 176.6 mm to (41.8, 20.5), turned to 90 degrees
- moved C43 176.4 mm to (41.3, 29.5), turned to -90 degrees
- moved D10 176.0 mm to (19.6, 7.50)
- moved Q2 176.0 mm to (16.6, 9.00)
- moved Q3 176.0 mm to (12.1, 6.50)
- moved Q4 176.0 mm to (12.1, 9.95)
- moved R20 176.0 mm to (16.6, 6.00)
- moved R22 176.0 mm to (9.06, 7.50)
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Connections:
- C20 pad 1: ADV7611_CVDD_1V8 -> ADV7611_PVDD_1V8
- C21 pad 1: ADV7611_CVDD_1V8 -> ADV7611_PVDD_1V8
- C26 pad 1: ADV7611_CVDD_1V8 -> ADV7611_DVDD_1V8
- C27 pad 1: ADV7611_CVDD_1V8 -> ADV7611_DVDD_1V8
- C28 pad 1: ADV7611_CVDD_1V8 -> ADV7611_DVDD_1V8
- C29 pad 1: ADV7611_CVDD_1V8 -> ADV7611_DVDD_1V8
- C30 pad 1: ADV7611_CVDD_1V8 -> ADV7611_DVDD_1V8
- C31 pad 1: ADV7611_CVDD_1V8 -> ADV7611_DVDD_1V8
- C32 pad 1: ADV7611_CVDD_1V8 -> ADV7611_DVDD_1V8
- C33 pad 1: ADV7611_CVDD_1V8 -> ADV7611_DVDD_1V8
- C35 pad 1: ADV7611_DVDDIO_3V3 -> +3V3
- C49 pad 1: ADV7611_CVDD_1V8 -> /Power/+1V8_ADV7611
- C52 pad 1: +1V2 -> +3V3
- C53 pad 1: +3V3 -> Net-(C53-Pad1)
- C53 pad 2: GND -> Net-(U13--)
- D12 pad 1: Net-(D12-K) -> +3V3
- D12 pad 2: Net-(D12-A) -> unconnected-(D12-NC-Pad2)
- J10 pad 9: /Data/ADV7611_LLC -> unconnected-(J10-Pin_9-Pad9)
- J12 pad 1: /Data/ICE40_RGB_0 -> unconnected-(J12-Pin_1-Pad1)
- J12 pad 10: unconnected-(J12-Pin_10-Pad10) -> MAC_VIDOUT_3V3_RP2350
- J12 pad 3: /Data/ICE40_RGB_1 -> unconnected-(J12-Pin_3-Pad3)
- J12 pad 7: /Data/ICE40_RGB_2 -> unconnected-(J12-Pin_7-Pad7)
- J12 pad 8: MAC_VIDOUT_3V3_RP2350 -> MAC_PWM_3V3_RP2350
- J5 pad 10: GND -> /Power/J5_GND
- J5 pad 11: GND -> /Power/J5_GND
- J5 pad 12: GND -> /Power/J5_GND
- J5 pad 13: GND -> /Power/J5_GND
- J5 pad 14: GND -> /Power/J5_GND
- J5 pad 6: /Power/MAC_VIDOUT -> /Power/MAC_VIDOUT_5V
- J5 pad 9: /Power/MAC_PWM -> /Power/MAC_PWM_5V
- J8 pad 1: /Data/ADV7611_Y7 -> /Data/ADV7611_Y6
- J8 pad 10: /Data/ADV7611_Y0 -> /Data/ADV7611_Y1
- J8 pad 2: /Data/ADV7611_Y3 -> /Data/ADV7611_Y7
- J8 pad 3: /Data/ADV7611_Y6 -> /Data/ADV7611_Y4
- J8 pad 4: /Data/ADV7611_Y2 -> /Data/ADV7611_Y5
- J8 pad 7: /Data/ADV7611_Y5 -> /Data/ADV7611_Y2
- J8 pad 8: /Data/ADV7611_Y1 -> /Data/ADV7611_Y3
- J8 pad 9: /Data/ADV7611_Y4 -> /Data/ADV7611_Y0
- J9 pad 2: /Data/ADV7611_CB3CR3 -> /Data/ADV7611_CB6CR6
- J9 pad 3: /Data/ADV7611_CB6CR6 -> /Data/ADV7611_CB5CR5
- J9 pad 4: /Data/ADV7611_CB2CR2 -> /Data/ADV7611_CB4CR4
- J9 pad 7: /Data/ADV7611_CB5CR5 -> /Data/ADV7611_CB3CR3
- J9 pad 8: /Data/ADV7611_CB1CR1 -> /Data/ADV7611_CB2CR2
- J9 pad 9: /Data/ADV7611_CB4CR4 -> /Data/ADV7611_CB1CR1
- R26 pad 1: /Data/ICE40_RESET_L -> Net-(D12-K)
- R26 pad 2: GND -> /Data/HDMI_CEC
- R31 pad 1: +3V3 -> ADV7611_DVDDIO_3V3
- R31 pad 2: Net-(U7-EN) -> /Data/ADV7611_INT1
- R58 pad 1: /Power/MAC_VSYNC_3V3_RP2350 -> MAC_VSYNC_3V3_RP2350
- R59 pad 1: /Power/MAC_VSYNC_3V3_ICE40 -> Net-(U2-B1Y)
- R59 pad 2: /Power/MAC_VSYNC_3V3 -> /Power/MAC_VSYNC_5V
- R60 pad 1: /Power/MAC_HSYNC_3V3_RP2350 -> MAC_HSYNC_3V3_RP2350
- R61 pad 1: /Power/MAC_HSYNC_3V3_ICE40 -> Net-(U2-B2Y)
- R61 pad 2: /Power/MAC_HSYNC_3V3 -> /Power/MAC_HSYNC_5V
- R62 pad 1: /Power/MAC_VIDOUT_3V3_RP2350 -> MAC_VIDOUT_3V3_RP2350
- R69 pad 1: /Power/MAC_VIDOUT_5V -> /Power/MAC_VIDOUT
- R69 pad 2: /Power/MAC_VIDOUT -> /Power/MAC_VIDOUT_5V
- R75 pad 2: Net-(U9-~{CE}) -> /Power/5V_MAC_ST_L
- U1 pad 24: ADV7611_CVDD_1V8 -> ADV7611_DVDD_1V8
- U1 pad 40: ADV7611_CVDD_1V8 -> ADV7611_DVDD_1V8
- U1 pad 48: /Data/I2S_ADV7611_TDM -> I2S_ADV7611_DOUT
- U1 pad 49: /Data/I2S_ADV7611_SCLK -> I2S_ADV7611_SCLK
- U1 pad 50: /Data/I2S_ADV7611_LRCLK -> I2S_ADV7611_LRCLK
- U1 pad 51: /Data/I2S_ADV7611_MCLK -> Net-(U1-MCLK/INT2)
- U1 pad 52: ADV7611_CVDD_1V8 -> ADV7611_DVDD_1V8
- U1 pad 57: ADV7611_CVDD_1V8 -> ADV7611_PVDD_1V8
- U1 pad 60: ADV7611_CVDD_1V8 -> ADV7611_DVDD_1V8
- U2 pad 10: unconnected-(U2-B4Y-Pad10) -> Net-(U2-B4Y)
- U2 pad 11: /Power/MAC_VIDOUT_5V -> Net-(U2-B3Y)
- U2 pad 12: /Power/MAC_HSYNC_5V -> Net-(U2-B2Y)
- U2 pad 13: /Power/MAC_VSYNC_5V -> Net-(U2-B1Y)
- U2 pad 4: /Power/MAC_VIDOUT_3V3 -> /Power/MAC_PWM_3V3
- U2 pad 5: unconnected-(U2-A4-Pad5) -> /Power/MAC_VIDOUT_3V3
- U3 pad 21: /Data/ICE40_CLK_FROM_RP2350 -> unconnected-(U3-GPIO21-Pad21)
- U3 pad 42: /Data/RP2350_ICE40_GPIO -> unconnected-(U3-GPIO33-Pad42)
- U3 pad 43: /Data/ICE40_RESET_L -> unconnected-(U3-GPIO34-Pad43)
- U3 pad 44: /Data/ICE40_DONE -> unconnected-(U3-GPIO35-Pad44)
- U3 pad 45: /Data/SPI_ICE40_SO -> unconnected-(U3-GPIO36-Pad45)
- U3 pad 46: /Data/SPI_ICE40_CS_L -> unconnected-(U3-GPIO37-Pad46)
- U3 pad 47: /Data/SPI_ICE40_SCK -> unconnected-(U3-GPIO38-Pad47)
- U3 pad 48: /Data/SPI_ICE40_SI -> unconnected-(U3-GPIO39-Pad48)
- U3 pad 50: /Data/UART_RP2350_RX -> +3V3
- U3 pad 52: unconnected-(U3-GPIO41/ADC1-Pad52) -> /Data/UART_RP2350_RX
- U3 pad 6: unconnected-(U3-GPIO8-Pad6) -> MAC_VSYNC_3V3_RP2350
- U3 pad 60: unconnected-(U3-IOVDD-Pad60) -> +3V3
- U3 pad 7: MAC_VSYNC_3V3_RP2350 -> MAC_HSYNC_3V3_RP2350
- U3 pad 8: MAC_HSYNC_3V3_RP2350 -> MAC_PWM_3V3_RP2350
- U6 pad 2: ADV7611_CVDD_1V8 -> /Power/+1V8_ADV7611
- U9 pad 3: Net-(U9-~{CE}) -> /Power/5V_MAC_ST_L
Routing:
- net +5V: track 0.00 -> 395.3 mm, vias 0 -> 21
- net I2S_ADV7611_SCLK: track 0.00 -> 126.4 mm, vias 0 -> 2
- net /Data/ADV7611_RESET_L: track 0.00 -> 118.5 mm, vias 0 -> 4
- net /Data/I2C_ADV7611_SDA: track 0.00 -> 118.2 mm, vias 0 -> 2
- net I2S_ADV7611_LRCLK: track 0.00 -> 118.1 mm, vias 0 -> 2
- net I2S_ADV7611_DOUT: track 0.00 -> 113.5 mm, vias 0 -> 2
- net /Data/ADV7611_INT1: track 0.00 -> 113.0 mm, vias 0 -> 4
- net /Data/I2C_ADV7611_SCL: track 0.00 -> 111.5 mm, vias 0 -> 2
- net ADV7611_DVDD_1V8: track 0.00 -> 110.1 mm, vias 0 -> 4
- net +5V_MAC: track 0.00 -> 97.5 mm, vias 0 -> 2
- net /Data/USB2_D_R_P: track 0.00 -> 86.6 mm
- net /Data/USB2_D_R_N: track 0.00 -> 85.7 mm
- net /Power/5V_MAC_ST_L: track 0.00 -> 78.5 mm, vias 0 -> 4
- net +3V3: track 0.00 -> 76.8 mm, vias 0 -> 41
- net ADV7611_DVDDIO_3V3: track 0.00 -> 76.7 mm, vias 0 -> 12
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- added copper zone on In2.Cu, net +1V1
- added copper zone on B.Cu, net +3V3
- added copper zone on F.Cu, net +3V3
- added copper zone on In2.Cu, net +3V3
- added copper zone on F.Cu, net +5V
- added copper zone on F.Cu, net +5V_USB
- added copper zone on In2.Cu, net /Power/+1V8_ADV7611
- added copper zone on B.Cu, net /Power/J5_GND
- added copper zone on F.Cu, net /Power/J5_GND
- added copper zone on In1.Cu, net /Power/J5_GND
- added copper zone on In2.Cu, net /Power/J5_GND
- added copper zone on In2.Cu, net ADV7611_CVDD_1V8
- added copper zone on F.Cu, net ADV7611_DVDDIO_3V3
- added copper zone on In2.Cu, net ADV7611_DVDDIO_3V3
- added copper zone on B.Cu, net GND
- added copper zone on F.Cu, net GND
- added copper zone on In1.Cu, net GND
- added copper zone on In2.Cu, net GND
Other:
- board size 4.5 x 13.4 mm -> 137.4 x 64 mm
- copper layers 2 -> 4
- board text added: "Spool Labs"

Commit message: near prod ready
Parts:
- removed D1, D2: LED, LED_SMD:LED_0805_2012Metric_Pad1.15x1.40mm_HandSolder
- added C54: 10uF, Capacitor_SMD:C_0805_2012Metric_Pad1.18x1.45mm_HandSolder, F.Cu at (31.0, 39.6)
- added C55: 10uF, Capacitor_SMD:C_0805_2012Metric_Pad1.18x1.45mm_HandSolder, F.Cu at (24.2, 34.5)
- added C56: 10uF, Capacitor_SMD:C_0805_2012Metric_Pad1.18x1.45mm_HandSolder, F.Cu at (34.5, 11.2)
- added C57: 10uF, Capacitor_SMD:C_0805_2012Metric_Pad1.18x1.45mm_HandSolder, F.Cu at (33.2, 36.0)
- added C58: 10uF, Capacitor_SMD:C_0805_2012Metric_Pad1.18x1.45mm_HandSolder, F.Cu at (18.0, 32.8)
- added D13: Red, LED_SMD:LED_0805_2012Metric_Pad1.15x1.40mm_HandSolder, F.Cu at (37.9, 58.2)
- added D14: Red, LED_SMD:LED_0805_2012Metric_Pad1.15x1.40mm_HandSolder, F.Cu at (56.5, 57.8)
- added FB4: BLM18KG601SN1D, mac-vintage-hdmi:L_0603_1608Metric_Pad1.05x0.95mm_HandSolder, F.Cu at (35.2, 38.0)
- added FB5: BLM18KG601SN1D, mac-vintage-hdmi:L_0603_1608Metric_Pad1.05x0.95mm_HandSolder, F.Cu at (18.0, 31.0)
- added R45: 33, Resistor_SMD:R_0402_1005Metric_Pad0.72x0.64mm_HandSolder, F.Cu at (42.5, 12.8)
- added R46: 33, Resistor_SMD:R_0402_1005Metric_Pad0.72x0.64mm_HandSolder, F.Cu at (43.6, 12.8)
- added R47: 33, Resistor_SMD:R_0402_1005Metric_Pad0.72x0.64mm_HandSolder, F.Cu at (41.4, 12.8)
- added R85: 0, Resistor_SMD:R_0805_2012Metric_Pad1.20x1.40mm_HandSolder, F.Cu at (117.4, 55.0)
- added R86: 0, Resistor_SMD:R_0805_2012Metric_Pad1.20x1.40mm_HandSolder, F.Cu at (117.4, 57.2)
- added R87: 0, Resistor_SMD:R_0805_2012Metric_Pad1.20x1.40mm_HandSolder, F.Cu at (117.4, 59.2)
- C13, C14: footprint Capacitor_SMD:C_0805_2012Metric_Pad1.18x1.45mm_HandSolder -> mac-vintage-hdmi:generic_capc1005x50_wide
- D10, D11, D4, D5, D6: value LED -> Green
- D15, D16: value LED -> Yellow
- D3: value LED -> Red
- R1: footprint Resistor_SMD:R_0805_2012Metric_Pad1.20x1.40mm_HandSolder -> Resistor_SMD:R_0402_1005Metric_Pad0.72x0.64mm_HandSolder
- R14, R7: value 1K -> 1k
- U12: value PT8211-S -> TM8211-TA2302
- moved R30 17.8 mm to (52.6, 39.6)
- moved R32 17.4 mm to (52.6, 38.2)
- moved R34 17.2 mm to (52.5, 36.8)
- moved R36 16.7 mm to (52.5, 35.5)
- moved R38 16.6 mm to (52.5, 33.9)
- moved R40 16.4 mm to (52.5, 32.7)
- moved R42 16.3 mm to (52.5, 31.3)
- moved R44 16.2 mm to (52.7, 30.0)
- moved C14 5.03 mm to (85.2, 40.2)
- moved C13 4.71 mm to (85.2, 39.5), turned to 180 degrees
- moved D6 4.25 mm to (80.2, 4.25), turned to 0 degrees
- moved R76 3.02 mm to (117.4, 52.8), turned to 0 degrees
- moved C49 2.80 mm to (50.1, 41.8)
- moved U6 2.80 mm to (50.3, 46.5)
- moved TP4 2.50 mm to (35.0, 6.50)
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Connections:
- C34 pad 1: ADV7611_DVDDIO_3V3 -> ADV7611_TVDD_3V3
- C36 pad 1: ADV7611_DVDDIO_3V3 -> ADV7611_TVDD_3V3
- C37 pad 1: ADV7611_DVDDIO_3V3 -> ADV7611_TVDD_3V3
- C38 pad 1: ADV7611_DVDDIO_3V3 -> ADV7611_TVDD_3V3
- C39 pad 1: ADV7611_DVDDIO_3V3 -> ADV7611_TVDD_3V3
- C47 pad 1: ADV7611_DVDDIO_3V3 -> /Power/+3V3_ADV7611
- C48 pad 1: ADV7611_DVDDIO_3V3 -> /Power/+3V3_ADV7611
- C83 pad 1: ADV7611_DVDDIO_3V3 -> ADV7611_TVDD_3V3
- J8 pad 1: /Data/ADV7611_Y6 -> /Data/ADV7611_Y6_RP2350
- J8 pad 10: /Data/ADV7611_Y1 -> /Data/ADV7611_Y1_RP2350
- J8 pad 2: /Data/ADV7611_Y7 -> /Data/ADV7611_Y7_RP2350
- J8 pad 3: /Data/ADV7611_Y4 -> /Data/ADV7611_Y4_RP2350
- J8 pad 4: /Data/ADV7611_Y5 -> /Data/ADV7611_Y5_RP2350
- J8 pad 7: /Data/ADV7611_Y2 -> /Data/ADV7611_Y2_RP2350
- J8 pad 8: /Data/ADV7611_Y3 -> /Data/ADV7611_Y3_RP2350
- J8 pad 9: /Data/ADV7611_Y0 -> /Data/ADV7611_Y0_RP2350
- L2 pad 1: Net-(U3-VREG_LX) -> +1V1
- L2 pad 2: +1V1 -> Net-(U3-VREG_LX)
- U1 pad 11: ADV7611_DVDDIO_3V3 -> ADV7611_TVDD_3V3
- U1 pad 48: I2S_ADV7611_DOUT -> /Data/I2S_ADV7611_DOUT_R
- U1 pad 49: I2S_ADV7611_SCLK -> /Data/I2S_ADV7611_SCLK_R
- U1 pad 5: ADV7611_DVDDIO_3V3 -> ADV7611_TVDD_3V3
- U1 pad 50: I2S_ADV7611_LRCLK -> /Data/I2S_ADV7611_LRCLK_R
- U1 pad 8: ADV7611_DVDDIO_3V3 -> ADV7611_TVDD_3V3
- U5 pad 2: ADV7611_DVDDIO_3V3 -> /Power/+3V3_ADV7611
- U6 pad 3: ADV7611_DVDDIO_3V3 -> /Power/+3V3_ADV7611
Routing:
- net ADV7611_TVDD_3V3: track 0.00 -> 37.0 mm, vias 0 -> 4
- net ADV7611_DVDDIO_3V3: track 76.7 -> 52.6 mm, vias 12 -> 7
- net /Data/ADV7611_Y0_RP2350: track 25.8 -> 45.8 mm
- net /Data/ADV7611_Y5_RP2350: track 23.2 -> 43.0 mm
- net /Data/ADV7611_Y1_RP2350: track 25.7 -> 45.5 mm
- net /Data/ADV7611_Y2_RP2350: track 24.5 -> 44.0 mm
- net /Data/ADV7611_Y6: track 42.7 -> 23.3 mm
- net /Data/ADV7611_Y7: track 43.8 -> 24.5 mm
- net /Data/ADV7611_Y4: track 40.3 -> 21.0 mm
- net /Data/ADV7611_Y5: track 40.6 -> 22.4 mm
- net /Data/ADV7611_Y2: track 36.8 -> 18.8 mm
- net /Data/ADV7611_Y3: track 37.7 -> 19.8 mm
- net /Data/ADV7611_Y7_RP2350: track 25.0 -> 42.8 mm
- net /Data/ADV7611_Y1: track 35.7 -> 17.9 mm
- net /Data/ADV7611_Y3_RP2350: track 25.1 -> 42.7 mm
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- added copper zone on B.Cu, net /Power/+3V3_ADV7611
- added copper zone on F.Cu, net /Power/+3V3_ADV7611
- added copper zone on F.Cu, net Net-(U3-VREG_LX)
- removed copper zone on F.Cu, net ADV7611_DVDDIO_3V3
Other:
- board text added: "mac-hdmi-adapter rev1.0"
- board text added: "spool labs"
- board text removed: "Spool Labs"

Commit message: added production export
Parts:
- C1, C10, C2, C3, C35, C4, C5, C52, C6, C7, C8, C9: value 100n -> 100nF
- C20, C23, C25, C27, C29, C31, C33, C37, C39, C41, C43, C45, C69, C70, C73, C75, C80, C83, C85: value 0.1uF -> 100nF
- D7, D8: value RCLAMP0524PA -> RCLAMP0524PATCT
- J6: value Conn_01x02 -> HX PZ2.54-1x2P ZZ; footprint mac-vintage-hdmi:PinHeader_1x02_P2.54mm_Vertical_SMD_Pin1Left -> mac-vintage-hdmi:PinHeader_1x02_P2.54mm_Vertical
- R10, R12, R13, R15, R20, R23, R73, R74, R8: value 5.1k -> 2.7k
- R9: value 5.1k -> 1k
- U1: value ADV7611 -> ADV7611BSWZ
- moved J6 2.09 mm to (58.8, 46.7)
Routing:
- net /Data/ADV7611_LLC: track 42.5 -> 41.3 mm
Other:
- board text added: "IMPEDANCE CONTROL TABLE"
- board text added: "NOTES: 1. Target impedances are from the KiCad tuning profiles. Fabricator may adjust trace width and spacing to meet target impedance. 2. Stackup: 4 layers, 1.6 mm (JLC04161H-7628). Cu L1/L4 35 um, L2/L3 15.2 um. L1-L2 and L3-L4: 7628 prepreg 0.2104 mm (Er 4.4). L2-L3: core 1.065 mm (Er 4.43). Solder mask 15 um (Er 3.8). 3. Coplanar rows: GND pour on the signal layer is 0.3 mm (11.81 mil) from t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"
