File: mac-vintage-hdmi/mac-vintage-hdmi.kicad_sch (KiCad schematic)
At the start: 112 parts, among them J1 HDMI_A, J10 Conn_02x05_Odd_Even, J11 Conn_02x05_Odd_Even, J12 Conn_02x05_Odd_Even, J3 BM03B-SRSS-TB, J4 BM03B-SRSS-TB, J8 Conn_02x05_Odd_Even, J9 Conn_02x05_Odd_Even, Q10 BSS123LT1, Q2 BSS123LT1, Q3 BSS123LT1, Q4 BSS123LT1, Q5 BSS123LT1, Q6 BSS123LT1, Q7 BSS123LT1, Q8 BSS123LT1, Q9 BSS123LT1, SW1 434133025816, SW2 434133025816, SW3 434133025816, U1 ADV7611, U3 RP2354B, U8 ICE40UP5K-SG48I, Y1 ABM8-272-T3, Y2 ABM8-28.63636MHZ-B2-T

Commit message: ready for design review
Parts:
- removed C15, C16, C56, C58, C60, C61, C63, C66: 100n, Capacitor_SMD:C_0402_1005Metric_Pad0.74x0.62mm_HandSolder, symbol Device:C
- removed C54, C55, C57, C59, C62, C64, C65: 4.7uF, Capacitor_SMD:C_0805_2012Metric_Pad1.18x1.45mm_HandSolder, symbol Device:C
- removed D12: LED, LED_SMD:LED_0805_2012Metric_Pad1.15x1.40mm_HandSolder, symbol Device:LED
- removed D13: MHPA1010RGBDT, mac-vintage-hdmi:LED_RGB_Meihua_MHPA1010RGBDT_1x1mm, symbol mac-vintage-hdmi:MHPA1010RGBDT
- removed J11: Conn_02x05_Odd_Even, mac-vintage-hdmi:PinHeader_2x05_P2.54mm_Vertical_SMD, symbol mac-vintage-hdmi:Conn_02x05_Odd_Even
- removed L1: 3.3uH, Inductor_SMD:L_0805_2012Metric_Pad1.05x1.20mm_HandSolder, symbol Device:L
- removed Q7, Q8: BSS123LT1, mac-vintage-hdmi:SOT-23, symbol mac-vintage-hdmi:BSS123LT1
- removed R16: 10k, Resistor_SMD:R_0805_2012Metric_Pad1.20x1.40mm_HandSolder, symbol Device:R_US
- removed R27: 100k, Resistor_SMD:R_0805_2012Metric_Pad1.20x1.40mm_HandSolder, symbol Device:R_US
- removed R28: 5.1k, Resistor_SMD:R_0805_2012Metric_Pad1.20x1.40mm_HandSolder, symbol Device:R_US
- removed R37: 100, Resistor_SMD:R_01005_0402Metric_Pad0.57x0.30mm_HandSolder, symbol Device:R_US
- removed R45, R46, R47, R48, R49, R50, R51, R52, R53, R54, R55, R57: 0, Resistor_SMD:R_01005_0402Metric_Pad0.57x0.30mm_HandSolder, symbol Device:R_US
- removed SW3: 434133025816, mac-vintage-hdmi:SW_Push_1P1T_NO_Vertical_Wuerth_434133025816, symbol mac-vintage-hdmi:434133025816
- removed U8: ICE40UP5K-SG48I, mac-vintage-hdmi:QFN-48-1EP_7x7mm_P0.5mm_EP5.3x5.3mm, symbol mac-vintage-hdmi:ICE40UP5K-SG48I
- added D12: MA3X704A, mac-vintage-hdmi:SC-59, symbol mac-vintage-hdmi:MA3X704A
- added J6: Conn_01x02, mac-vintage-hdmi:PinHeader_1x02_P2.54mm_Vertical_SMD_Pin1Left, symbol mac-vintage-hdmi:Conn_01x02
- added L2: AOTA-B201610S3R3-101-T, mac-vintage-hdmi:L_Abracon_AOTA-B201610S3R3-101-T_2.0x1.6mm, symbol mac-vintage-hdmi:AOTA-B201610S3R3-101-T
- added R31: 2.7k, Resistor_SMD:R_0805_2012Metric_Pad1.20x1.40mm_HandSolder, symbol Device:R_US
- added TP4: TestPoint, TestPoint:TestPoint_Pad_2.0x2.0mm, symbol Connector:TestPoint
- R26: value 100k -> 27k
- R30, R32, R34, R36, R38, R39, R40, R41, R42, R43, R44, R56: value 0 -> 33; footprint Resistor_SMD:R_01005_0402Metric_Pad0.57x0.30mm_HandSolder -> Resistor_SMD:R_0402_1005Metric_Pad0.72x0.64mm_HandSolder
Connections:
- net +1V1: now also L2.2
- net +3V3: now also U3.50 (IOVDD), U3.60 (IOVDD), D12.1 (A)
- net ADV7611_CB1CR1: now also J9.9 (Pin_9); no longer J9.8 (Pin_8)
- net ADV7611_CB2CR2: now also J9.8 (Pin_8); no longer J9.4 (Pin_4)
- net ADV7611_CB3CR3: now also J9.7 (Pin_7); no longer J9.2 (Pin_2)
- net ADV7611_CB4CR4: now also J9.4 (Pin_4); no longer J9.9 (Pin_9)
- net ADV7611_CB5CR5: now also J9.3 (Pin_3); no longer J9.7 (Pin_7)
- net ADV7611_CB6CR6: now also J9.2 (Pin_2); no longer J9.3 (Pin_3)
- net ADV7611_DVDDIO_3V3: now also R31.1
- net ADV7611_INT1: now also R31.2
- net ADV7611_LLC: now also J6.1 (Pin_1); no longer J10.9 (Pin_9)
- net ADV7611_Y0: now also J8.9 (Pin_9); no longer J8.10 (Pin_10)
- net ADV7611_Y1: now also J8.10 (Pin_10); no longer J8.8 (Pin_8)
- net ADV7611_Y2: now also J8.7 (Pin_7); no longer J8.4 (Pin_4)
- net ADV7611_Y3: now also J8.8 (Pin_8); no longer J8.2 (Pin_2)
- net ADV7611_Y4: now also J8.3 (Pin_3); no longer J8.9 (Pin_9)
- net ADV7611_Y5: now also J8.4 (Pin_4); no longer J8.7 (Pin_7)
- net ADV7611_Y6: now also J8.1 (Pin_1); no longer J8.3 (Pin_3)
- net ADV7611_Y7: now also J8.2 (Pin_2); no longer J8.1 (Pin_1)
- net GND: now also J6.2 (Pin_2); no longer R26.2
- net HDMI_CEC: now also R26.2
- net MAC_HSYNC_3V3_RP2350: now also U3.7 (GPIO9); no longer U3.8 (GPIO10)
- net MAC_VIDOUT_3V3_RP2350: now also J12.10 (Pin_10); no longer J12.8 (Pin_8)
- net MAC_VSYNC_3V3_RP2350: now also U3.6 (GPIO8); no longer U3.7 (GPIO9)
- net UART_RP2350_RX: now also U3.52 (GPIO41/ADC1); no longer U3.50 (IOVDD)
- net at U3.63 (VREG_LX): now also L2.1
- net I2S_ADV7611_MCLK: no longer names the net of U1.51 (MCLK/INT2)
- net I2S_ADV7611_MCLK: now also TP4.1
- net I2S_ADV7611_TDM renamed I2S_ADV7611_DOUT
- net ICE40_CLK_FROM_RP2350: no longer names the net of U3.21 (GPIO21)
- net ICE40_DONE: no longer names the net of U3.44 (GPIO35)
- net ICE40_RESET_L: no longer names the net of R26.1
- net ICE40_RESET_L: now also D12.3 (K); no longer U3.43 (GPIO34)
- net ICE40_RGB_0: no longer names the net of J12.1 (Pin_1)
- net ICE40_RGB_1: no longer names the net of J12.3 (Pin_3)
- net ICE40_RGB_2: no longer names the net of J12.7 (Pin_7)
- net RP2350_ICE40_GPIO: no longer names the net of U3.42 (GPIO33)
- net SPI_ICE40_CS_L: no longer names the net of U3.46 (GPIO37)
- net SPI_ICE40_SCK: no longer names the net of U3.47 (GPIO38)
- net SPI_ICE40_SI: no longer names the net of U3.48 (GPIO39)
- net SPI_ICE40_SO: no longer names the net of U3.45 (GPIO36)
- new net MAC_PWM_3V3_RP2350: J12.8 (Pin_8), U3.8 (GPIO10)
- no-connect marks 44 -> 49
Other:
- note added: "PWM4A/PIO1"
- note removed: "CLOCK GPOUT0"
- note removed: "ICE40"
- note removed: "ICE40 LEDs and Buttons"
- moved on the sheet: C12, D10, D11, J12, Q2, Q3, Q4, Q5, Q6, R1, R18, R19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

Commit message: near prod ready
Parts:
- added R45, R46, R47: 33, Resistor_SMD:R_0402_1005Metric_Pad0.72x0.64mm_HandSolder, symbol Device:R_US
- C13, C14: footprint Capacitor_SMD:C_0805_2012Metric_Pad1.18x1.45mm_HandSolder -> mac-vintage-hdmi:generic_capc1005x50_wide
- D10, D11, D4, D5, D6: value LED -> Green; MPN (none) -> LG R971-KN-1-0-20-R18
- R1: footprint Resistor_SMD:R_0805_2012Metric_Pad1.20x1.40mm_HandSolder -> Resistor_SMD:R_0402_1005Metric_Pad0.72x0.64mm_HandSolder
- R14, R7: value 1K -> 1k
Connections:
- net +1V1: now also L2.1; no longer L2.2
- net ADV7611_Y0: no longer J8.9 (Pin_9)
- net ADV7611_Y0_RP2350: now also J8.9 (Pin_9)
- net ADV7611_Y1: no longer J8.10 (Pin_10)
- net ADV7611_Y1_RP2350: now also J8.10 (Pin_10)
- net ADV7611_Y2: no longer J8.7 (Pin_7)
- net ADV7611_Y2_RP2350: now also J8.7 (Pin_7)
- net ADV7611_Y3: no longer J8.8 (Pin_8)
- net ADV7611_Y3_RP2350: now also J8.8 (Pin_8)
- net ADV7611_Y4: no longer J8.3 (Pin_3)
- net ADV7611_Y4_RP2350: now also J8.3 (Pin_3)
- net ADV7611_Y5: no longer J8.4 (Pin_4)
- net ADV7611_Y5_RP2350: now also J8.4 (Pin_4)
- net ADV7611_Y6: no longer J8.1 (Pin_1)
- net ADV7611_Y6_RP2350: now also J8.1 (Pin_1)
- net ADV7611_Y7: no longer J8.2 (Pin_2)
- net ADV7611_Y7_RP2350: now also J8.2 (Pin_2)
- net I2S_ADV7611_DOUT: now also R45.2; no longer U1.48 (AP)
- net I2S_ADV7611_LRCLK: now also R47.2; no longer U1.50 (LRCLK)
- net I2S_ADV7611_SCLK: now also R46.2; no longer U1.49 (SCLK/INT2)
- net at U3.63 (VREG_LX): now also L2.2; no longer L2.1
- new net I2S_ADV7611_DOUT_R: R45.1, U1.48 (AP)
- new net I2S_ADV7611_LRCLK_R: R47.1, U1.50 (LRCLK)
- new net I2S_ADV7611_SCLK_R: R46.1, U1.49 (SCLK/INT2)
Other:
- note added: "L2 alternates on LCSC (unmarked; orientation will be random): C5832345 Changjiang FTC201610S3R3MBCA C41405891 YJYCOIN YSMC201612H-3R3MB* C39846627 XR XRIM201612S3R3MBCA* C48945398 ZE ZET-CORE-201608ST3R3MBCA *1.2 mm tall. All meet RP2350 DS §6.3.8.2: DCR ≤250mΩ, Isat ≥1.5A."
- note removed: "todo: figure out audio solution just break out signals to another possible board unless there is an easy audio solution that can fit within current limits What does the sound signal input into the display board, need?"

Commit message: added production export
Parts:
- D12: LCSC_Alt (none) -> C232585
- D7, D8: value RCLAMP0524PA -> RCLAMP0524PATCT; symbol mac-vintage-hdmi:RCLAMP0524PA -> mac-vintage-hdmi:RCLAMP0524PATCT
- J10, J12, J8, J9: LCSC_Alt (none) -> C3294463
- J6: value Conn_01x02 -> HX PZ2.54-1x2P ZZ; footprint mac-vintage-hdmi:PinHeader_1x02_P2.54mm_Vertical_SMD_Pin1Left -> mac-vintage-hdmi:PinHeader_1x02_P2.54mm_Vertical; symbol mac-vintage-hdmi:Conn_01x02 -> mac-vintage-hdmi:HX_PZ2.54-1x2P_ZZ
- R12, R13, R15, R20, R23: value 5.1k -> 2.7k
- SW1, SW2: LCSC_Alt (none) -> C116501
- U1: value ADV7611 -> ADV7611BSWZ; symbol mac-vintage-hdmi:ADV7611 -> mac-vintage-hdmi:ADV7611BSWZ
Changed lines of the file:
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@@
 		)
 		(property "Value" "Green"
-			(at 198.374 277.368 90)
+			(at 197.104 277.114 90)
 			(show_name no)
 			(do_not_autoplace no)
@@
 	)
 	(symbol
-		(lib_id "mac-vintage-hdmi:RCLAMP0524PA")
+		(lib_id "mac-vintage-hdmi:RCLAMP0524PATCT")
 		(at 90.17 38.1 0)
 		(unit 1)
@@
 			)
 		)
-		(property "Value" "RCLAMP0524PA"
+		(property "Value" "RCLAMP0524PATCT"
 			(at 90.424 30.48 0)
 			(show_name no)
@@
 			)
 		)
-		(property "Value" "5.1k"
+		(property "Value" "2.7k"
 			(at 341.63 267.9699 0)
 			(show_name no)
@@
 			)
 		)
-		(property "Value" "5.1k"
+		(property "Value" "2.7k"
 			(at 396.24 270.5099 0)
 			(show_name no)
@@
 	)
 	(symbol
-		(lib_id "mac-vintage-hdmi:Conn_01x02")
+		(lib_id "mac-vintage-hdmi:HX_PZ2.54-1x2P_ZZ")
 		(at 341.63 389.89 0)
 		(unit 1)
@@
 			)
 		)
-		(property "Value" "Conn_01x02"
+		(property "Value" "HX PZ2.54-1x2P ZZ"
 			(at 344.17 392.4299 0)
 			(show_name no)
@@
 			)
 		)
-		(property "Footprint" "mac-vintage-hdmi:PinHeader_1x02_P2.54mm_Vertical_SMD_Pin1Left"
+		(property "Footprint" "mac-vintage-hdmi:PinHeader_1x02_P2.54mm_Vertical"
 			(at 341.63 389.89 0)
 			(hide yes)
@@
 			)
 		)
-		(property "Datasheet" ""
+		(property "Datasheet" "https://www.lcsc.com/datasheet/C32713268.pdf"
 			(at 341.63 389.89 0)
 			(hide yes)
@@
 			)
 		)
-		(property "Description" "Generic connector, single row, 01x02, script generated (kicad-library-utils/schlib/autogen/connector/)"
+		(property "Description" "Hanxia 1x02 2.54mm straight male pin header, through-hole, single row, 2.5mm insulator, 6mm mating pin, gold (LCSC C32713268)"
 			(at 341.63 389.89 0)
 			(hide yes)
@@
 	)
 	(symbol
-		(lib_id "mac-vintage-hdmi:ADV7611")
+		(lib_id "mac-vintage-hdmi:ADV7611BSWZ")
 		(at 173.99 97.79 0)
 		(unit 1)
@@
 			)
 		)
-		(property "Value" "ADV7611"
+		(property "Value" "ADV7611BSWZ"
 			(at 176.1333 151.13 0)
 			(show_name no)
@@
 	)
 	(symbol
-		(lib_id "mac-vintage-hdmi:RCLAMP0524PA")
+		(lib_id "mac-vintage-hdmi:RCLAMP0524PATCT")
 		(at 88.9 68.58 0)
 		(unit 1)
@@
 			)
 		)
-		(property "Value" "RCLAMP0524PA"
+		(property "Value" "RCLAMP0524PATCT"
 			(at 89.154 60.706 0)
 			(show_name no)
@@
 			)
 		)
-		(property "Value" "5.1k"
+		(property "Value" "2.7k"
 			(at 219.71 312.4199 0)
 			(show_name no)
@@
 			)
 		)
+		(property "LCSC_Alt" "C232585"
+			(at 69.85 129.54 0)
+			(hide yes)
+			(show_name no)
+			(do_not_autoplace no)
+			(effects
+				(font
+					(size 1.27 1.27)
+				)
+			)
+		)
 		(pin "3"
 		)
@@
 			)
 		)
+		(property "LCSC_Alt" "C3294463"
+			(at 374.65 378.46 0)
+			(hide yes)
+			(show_name no)
+			(do_not_autoplace no)
+			(effects
+				(font
+					(size 1.27 1.27)
+				)
+			)
+		)
 		(pin "1"
 		)
@@
 			)
 		)
+		(property "LCSC_Alt" "C3294463"
+			(at 293.37 379.73 0)
+			(hide yes)
+			(show_name no)
+			(do_not_autoplace no)
+			(effects
+				(font
+					(size 1.27 1.27)
+				)
+			)
+		)
 		(pin "1"
 		)
@@
 		(fields_autoplaced yes)
 		(property "Reference" "R13"
-			(at 201.93 266.6999 0)
+			(at 207.01 266.6999 0)
 			(show_name no)
 			(do_not_autoplace no)
@@
 					(size 1.27 1.27)
 				)
-				(justify left)
+				(justify right)
 			)
 		)
-		(property "Value" "5.1k"
-			(at 201.93 269.2399 0)
+		(property "Value" "2.7k"
+			(at 207.01 269.2399 0)
 			(show_name no)
 			(do_not_autoplace no)
@@
 					(size 1.27 1.27)
 				)
-				(justify left)
+				(justify right)
 			)
 		)
@@
 			)
 		)
+		(property "LCSC_Alt" "C116501"
+			(at 198.12 344.17 0)
+			(hide yes)
+			(show_name no)
+			(do_not_autoplace no)
+			(effects
+				(font
+					(size 1.27 1.27)
+				)
+			)
+		)
 		(pin "2"
 		)
@@
 			)
 		)
+		(property "LCSC_Alt" "C3294463"
+			(at 293.37 354.33 0)
+			(hide yes)
+			(show_name no)
+			(do_not_autoplace no)
+			(effects
+				(font
+					(size 1.27 1.27)
+				)
+			)
+		)
 		(pin "1"
 		)
@@
 			)
 		)
+		(property "LCSC_Alt" "C116501"
+			(at 184.15 300.99 0)
+			(hide yes)
+			(show_name no)
+			(do_not_autoplace no)
+			(effects
+				(font
+					(size 1.27 1.27)
+				)
+			)
+		)
 		(pin "2"
 		)
@@
 			)
 		)
+		(property "LCSC_Alt" "C3294463"
+			(at 374.65 353.06 0)
+			(hide yes)
+			(show_name no)
+			(do_not_autoplace no)
+			(effects
+				(font
+					(size 1.27 1.27)
+				)
+			)
+		)
 		(pin "1"
 		)
@@
 			)
 		)
-		(property "Value" "5.1k"
+		(property "Value" "2.7k"
 			(at 224.79 256.5399 0)
 			(show_name no)
