File: mac-vintage-hdmi/power.kicad_sch (KiCad schematic)
At the start: 89 parts, among them J2 USB_C_Receptacle_USB2.0_16P, J5 39-28-1143, Q1 Si2342DS, U10 LM66100DCKR, U2 TXU0104PWR, U4 NCP1117-3.3_SOT223, U5 NCP1117-3.3_SOT223, U6 NCP1117ST18T3G, U7 NCP115AMX120TCG, U9 LM66100DCKR

Commit message: more placement
Parts:
- R68: footprint Resistor_SMD:R_01005_0402Metric_Pad0.57x0.30mm_HandSolder -> Resistor_SMD:R_0805_2012Metric_Pad1.20x1.40mm_HandSolder
Connections:
- net +5V: now also R68.1; no longer R68.2
- net at U2.8 (OE): now also R68.2; no longer R68.1
Changed lines of the file:
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@@
-	(symbol
-		(lib_id "Device:R_US")
-		(at 223.52 242.57 180)
-		(unit 1)
-		(body_style 1)
-		(exclude_from_sim no)
-		(in_bom yes)
-		(on_board yes)
-		(in_pos_files yes)
-		(dnp no)
-		(property "Reference" "R68"
-			(at 220.98 239.268 0)
-			(show_name no)
-			(do_not_autoplace no)
-			(effects
-				(font
-					(size 1.27 1.27)
-				)
-			)
-		)
-		(property "Value" "0"
-			(at 222.25 246.38 0)
-			(show_name no)
-			(do_not_autoplace no)
-			(effects
-				(font
-					(size 1.27 1.27)
-				)
-			)
-		)
-		(property "Footprint" "Resistor_SMD:R_01005_0402Metric_Pad0.57x0.30mm_HandSolder"
-			(at 222.504 242.316 90)
-			(hide yes)
-			(show_name no)
-			(do_not_autoplace no)
-			(effects
-				(font
-					(size 1.27 1.27)
-				)
-			)
-		)
-		(property "Datasheet" ""
-			(at 223.52 242.57 0)
-			(hide yes)
-			(show_name no)
-			(do_not_autoplace no)
-			(effects
-				(font
-					(size 1.27 1.27)
-				)
-			)
-		)
-		(property "Description" "Resistor, US symbol"
-			(at 223.52 242.57 0)
-			(hide yes)
-			(show_name no)
-			(do_not_autoplace no)
-			(effects
-				(font
-					(size 1.27 1.27)
-				)
-			)
-		)
-		(pin "2"
-		)
-		(pin "1"
-		)
-		(instances
-			(project "mac-vintage-hdmi"
-				(path "/13e48c44-097d-4a9e-b5ad-c93c72414a8b"
-					(reference "R68")
-					(unit 1)
-				)
-			)
-		)
-	)
 	(symbol
 		(lib_id "Device:R_US")
@@
 					(unit 1)
 				)
+			)
+		)
+	)
+	(symbol
+		(lib_id "Device:R_US")
+		(at 223.52 242.57 0)
+		(mirror y)
+		(unit 1)
+		(body_style 1)
+		(exclude_from_sim no)
+		(in_bom yes)
+		(on_board yes)
+		(in_pos_files yes)
+		(dnp no)
+		(property "Reference" "R68"
+			(at 220.98 241.2999 0)
+			(show_name no)
+			(do_not_autoplace no)
+			(effects
+				(font
+					(size 1.27 1.27)
+				)
+				(justify left)
+			)
+		)
+		(property "Value" "0"
+			(at 220.98 243.8399 0)
+			(show_name no)
+			(do_not_autoplace no)
+			(effects
+				(font
+					(size 1.27 1.27)
+				)
+				(justify left)
+			)
+		)
+		(property "Footprint" "Resistor_SMD:R_0805_2012Metric_Pad1.20x1.40mm_HandSolder"
+			(at 222.504 242.824 90)
+			(hide yes)
+			(show_name no)
+			(do_not_autoplace no)
+			(effects
+				(font
+					(size 1.27 1.27)
+				)
+			)
+		)
+		(property "Datasheet" ""
+			(at 223.52 242.57 0)
+			(hide yes)
+			(show_name no)
+			(do_not_autoplace no)
+			(effects
+				(font
+					(size 1.27 1.27)
+				)
+			)
+		)
+		(property "Description" "Resistor, US symbol"
+			(at 223.52 242.57 0)
+			(hide yes)
+			(show_name no)
+			(do_not_autoplace no)
+			(effects
+				(font
+					(size 1.27 1.27)
+				)
+			)
+		)
+		(pin "2"
+		)
+		(pin "1"
+		)
+		(instances
+			(project "mac-vintage-hdmi"
+				(path "/13e48c44-097d-4a9e-b5ad-c93c72414a8b"
+					(reference "R68")
+					(unit 1)
+				)

Commit message: ready for design review
Parts:
- removed R31: 0, Resistor_SMD:R_0805_2012Metric_Pad1.20x1.40mm_HandSolder, symbol Device:R_US
- removed R63: 0, Resistor_SMD:R_01005_0402Metric_Pad0.57x0.30mm_HandSolder, symbol Device:R_US
- removed U7: NCP115AMX120TCG, Package_DFN_QFN:OnSemi_XDFN4-1EP_1.0x1.0mm_EP0.52x0.52mm, symbol Regulator_Linear:NCP115AMX120TCG
- added C73, C75, C80, C85: 0.1uF, Capacitor_SMD:C_0805_2012Metric_Pad1.18x1.45mm_HandSolder, symbol Device:C
- added C74, C77, C84: 47uF, Capacitor_SMD:C_1210_3225Metric_Pad1.33x2.70mm_HandSolder, symbol Device:C
- added C76, C79: 10uF, Capacitor_SMD:C_0805_2012Metric_Pad1.18x1.45mm_HandSolder, symbol Device:C
- added C78: 47nF, Capacitor_SMD:C_0805_2012Metric_Pad1.18x1.45mm_HandSolder, symbol Device:C
- added C81: 470pF, Capacitor_SMD:C_0805_2012Metric_Pad1.18x1.45mm_HandSolder, symbol Device:C
- added C82: 1nF, Capacitor_SMD:C_0805_2012Metric_Pad1.18x1.45mm_HandSolder, symbol Device:C
- added C83: 0.1uF, Capacitor_SMD:C_0402_1005Metric_Pad0.74x0.62mm_HandSolder, symbol Device:C
- added FB1, FB2, FB3: BLM18KG601SN1D, mac-vintage-hdmi:L_0603_1608Metric_Pad1.05x0.95mm_HandSolder, symbol mac-vintage-hdmi:BLM18KG601SN1D
- added R76: 0, Resistor_SMD:R_0805_2012Metric_Pad1.20x1.40mm_HandSolder, symbol Device:R_US
- added R77, R78, R81, R84: 0, Resistor_SMD:R_0402_1005Metric_Pad0.72x0.64mm_HandSolder, symbol Device:R_US
- added R79: 5.1k, Resistor_SMD:R_0805_2012Metric_Pad1.20x1.40mm_HandSolder, symbol Device:R_US
- added R80: 47, Resistor_SMD:R_0805_2012Metric_Pad1.20x1.40mm_HandSolder, symbol Device:R_US
- added R82: 13k, Resistor_SMD:R_0805_2012Metric_Pad1.20x1.40mm_HandSolder, symbol Device:R_US
- added R83: 8.2k, Resistor_SMD:R_0805_2012Metric_Pad1.20x1.40mm_HandSolder, symbol Device:R_US
- added RV1: PTV09A, mac-vintage-hdmi:Potentiometer_Bourns_PTV09A_RearMount, symbol mac-vintage-hdmi:PTV09A
- added TP5: TestPoint, TestPoint:TestPoint_Pad_2.0x2.0mm, symbol Connector:TestPoint
- added U11: LM386M-1, mac-vintage-hdmi:SOIC-8_3.9x4.9mm_P1.27mm, symbol mac-vintage-hdmi:LM386M-1
- added U12: PT8211-S, mac-vintage-hdmi:SOIC-8_3.9x4.9mm_P1.27mm, symbol mac-vintage-hdmi:PT8211-S
- added U13: TLV9061IDBVR, mac-vintage-hdmi:SOT-23-5, symbol mac-vintage-hdmi:TLV9061IDBVR
- C35: value 0.1uF -> 100n; footprint Capacitor_SMD:C_0805_2012Metric_Pad1.18x1.45mm_HandSolder -> Capacitor_SMD:C_0402_1005Metric_Pad0.74x0.62mm_HandSolder
- C37, C39: footprint Capacitor_SMD:C_0805_2012Metric_Pad1.18x1.45mm_HandSolder -> Capacitor_SMD:C_0402_1005Metric_Pad0.74x0.62mm_HandSolder
- C52: value 4.7uF -> 100n; footprint Capacitor_SMD:C_0805_2012Metric_Pad1.18x1.45mm_HandSolder -> Capacitor_SMD:C_0402_1005Metric_Pad0.74x0.62mm_HandSolder
- C53: value 4.7uF -> 10uF
- J2: value USB_C_Receptacle_USB2.0_16P -> TYPE-C-31-M-12; footprint Connector_USB:USB_C_Receptacle_Amphenol_12401948E412A -> mac-vintage-hdmi:USB_C_Receptacle_HRO_TYPE-C-31-M-12; symbol Connector:USB_C_Receptacle_USB2.0_16P -> mac-vintage-hdmi:TYPE-C-31-M-12
- R58, R60, R62, R69: footprint Resistor_SMD:R_01005_0402Metric_Pad0.57x0.30mm_HandSolder -> Resistor_SMD:R_0402_1005Metric_Pad0.72x0.64mm_HandSolder
- R59, R61: footprint Resistor_SMD:R_01005_0402Metric_Pad0.57x0.30mm_HandSolder -> Resistor_SMD:R_0402_1005Metric_Pad0.72x0.64mm_HandSolder; now fitted
- R64: footprint Resistor_SMD:R_01005_0402Metric_Pad0.57x0.30mm_HandSolder -> Resistor_SMD:R_0402_1005Metric_Pad0.72x0.64mm_HandSolder; now not fitted
- R75: value 0 -> 1k
- U6: footprint mac-vintage-hdmi:SOT-223 -> mac-vintage-hdmi:SOT-223-3_TabPin2
Connections:
- net +1V2 is gone; now on net +3V3: C52.1
- net +12V_MAC: now also C84.1, C85.2, U11.6 (V+)
- net +3V3: now also C35.1, C73.1, C74.1, U12.5 (VDD); no longer C53.1
- net +5V: now also C80.1, U13.5 (V+)
- net +5V_USB: now also J2.A4/B9 (VBUS), J2.B4/A9 (VBUS); no longer J2.A4 (VBUS), J2.A9 (VBUS), J2.B4 (VBUS), J2.B9 (VBUS)
- net 5V_MAC_ST_L: now also R75.2, U9.3 (~{CE})
- net ADV7611_CVDD_1V8: now also FB3.2; no longer C20.1, C21.1, C26.1, C27.1, C28.1, C29.1, C30.1, C31.1, C32.1, C33.1, C49.1, U6.2 (VO), U6.4 (VO)
- net ADV7611_DVDDIO_3V3: now also C83.1; no longer C35.1
- net GND: now also J2.A1/B12 (GND), J2.B1/A12 (GND), J2.S1 (SHIELD), J2.S2 (SHIELD), J2.S3 (SHIELD), J2.S4 (SHIELD), C73.2, C74.2, C76.1, C78.2, C80.2, C81.2, C83.2, C84.2, C85.1, R76.2, RV1.3, RV1.4 (MP), RV1.5 (MP), U11.2 (-), U11.4 (GND), U12.4 (GND), U13.2 (V-); no longer C53.2, J2.A1 (GND), J2.A12 (GND), J2.B1 (GND), J2.B12 (GND), J2.SH (SHIELD), J5.10 (Pin_10), J5.11 (Pin_11), J5.12 (Pin_12), J5.13 (Pin_13), J5.14 (Pin_14)
- net MAC_HSYNC_3V3: no longer R61.2
- net MAC_HSYNC_5V: now also R61.2; no longer U2.12 (B2Y)
- net MAC_SOUND: now also C77.1
- net MAC_VIDOUT: now also R69.1; no longer J5.6 (Pin_6), R69.2
- net MAC_VIDOUT_3V3: now also U2.5 (A4); no longer U2.4 (A3)
- net MAC_VIDOUT_5V: now also J5.6 (Pin_6), R69.2, R84.2; no longer R69.1, U2.11 (B3Y)
- net MAC_VSYNC_3V3: no longer R59.2
- net MAC_VSYNC_5V: now also R59.2; no longer U2.13 (B1Y)
- net at U2.10 (B4Y): now also R84.1
- net MAC_HSYNC_3V3_ICE40: no longer names the net of R61.1
- net MAC_HSYNC_3V3_ICE40: now also U2.12 (B2Y)
- net MAC_PWM renamed MAC_PWM_5V
- net MAC_PWM_5V: now also R78.2
- net MAC_VSYNC_3V3_ICE40: no longer names the net of R59.1
- net MAC_VSYNC_3V3_ICE40: now also U2.13 (B1Y)
- new net: C75.2, U11.1 (GAIN)
- new net: C79.1, U11.3 (+)
- new net: C77.2, R80.1, U11.5
- new net: C76.2, U11.7 (BYPASS)
- new net: R79.1, U11.8 (GAIN)
- new net: C79.2, RV1.2
- new net: R78.1, U2.11 (B3Y)
- new net: C53.2, C82.1, R81.2, U13.1, U13.4 (-)
- new net: C82.2, R82.2, R83.1
- new net: C81.1, R83.2, U13.3 (+)
- new net: C53.1, RV1.1
- new net: TP5.1, U12.8 (RCH)
- new net: R81.1, R82.1, U12.6 (LCH)
- new net: C78.1, R80.2
- new net: C75.1, R79.2
- new net +1V8_ADV7611: C49.1, FB1.1, FB2.1, FB3.1, U6.2 (VO)
- new net ADV7611_DVDD_1V8: C26.1, C27.1, C28.1, C29.1, C30.1, C31.1, C32.1, C33.1, FB2.2
- new net ADV7611_PVDD_1V8: C20.1, C21.1, FB1.2
- new net I2S_ADV7611_DOUT: U12.3 (DIN)
- new net I2S_ADV7611_LRCLK: U12.2 (WS)
- new net I2S_ADV7611_SCLK: U12.1 (BCK)
- new net J5_GND: J5.10 (Pin_10), J5.11 (Pin_11), J5.12 (Pin_12), J5.13 (Pin_13), J5.14 (Pin_14), R76.1
- new net MAC_PWM_3V3: R77.2, U2.4 (A3)
- new net MAC_PWM_3V3_RP2350: R77.1
- no-connect marks 2 -> 0
Other:
- note added: "Amp"
- note added: "Audio pipeline"
- note added: "Can put series resistors here if I want"
- note added: "Filter design from https://hackaday.io/project/199220-catchcam-speed-camera-detector/log/234486-designing-audio-circuitry"
- note added: "I2S DAC"
- note added: "Low-pass filter"
- note added: "todo: check each pin aginst actual real life connector"
- note removed: "ICE40 1.2V"
- note removed: "todo: check on ESD on HDMI port and USB port"
- note removed: "todo: decided on League Gothic as a font Alpine Labs oilstainlab"
- moved on the sheet: C49, R58, R60, R62, R75

Commit message: near prod ready
Parts:
- removed D1, D2: LED, LED_SMD:LED_0805_2012Metric_Pad1.15x1.40mm_HandSolder, symbol Device:LED
- added C54, C55, C56, C57, C58: 10uF, Capacitor_SMD:C_0805_2012Metric_Pad1.18x1.45mm_HandSolder, symbol Device:C
- added D13, D14: Red, LED_SMD:LED_0805_2012Metric_Pad1.15x1.40mm_HandSolder, symbol Device:LED
- added FB4, FB5: BLM18KG601SN1D, mac-vintage-hdmi:L_0603_1608Metric_Pad1.05x0.95mm_HandSolder, symbol mac-vintage-hdmi:BLM18KG601SN1D
- added R85, R86, R87: 0, Resistor_SMD:R_0805_2012Metric_Pad1.20x1.40mm_HandSolder, symbol Device:R_US
- D15, D16: value LED -> Yellow; MPN (none) -> LY R976-PS-36-0-20-R18
- D3: value LED -> Red; MPN (none) -> LS R976-NR-1-0-20-R18
- U12: value PT8211-S -> TM8211-TA2302; LCSC (none) -> C22381766
Connections:
- net ADV7611_CVDD_1V8: now also C55.1
- net ADV7611_DVDDIO_3V3: now also C57.1, FB4.2; no longer C34.1, C36.1, C37.1, C38.1, C39.1, C47.1, C48.1, C83.1, U5.2 (VO), U6.3 (VI)
- net ADV7611_DVDD_1V8: now also C54.1
- net ADV7611_PVDD_1V8: now also C56.1
- net GND: now also C54.2, C55.2, C56.2, C57.2, C58.2, D13.1 (K), D14.1 (K), R85.2, R86.2, R87.2
- net J5_GND: now also R85.1, R86.1, R87.1
- net at R8.2: now also D14.2 (A)
- net at R9.2: now also D13.2 (A)
- new net +3V3_ADV7611: C47.1, C48.1, FB4.1, FB5.1, U5.2 (VO), U6.3 (VI)
- new net ADV7611_TVDD_3V3: C34.1, C36.1, C37.1, C38.1, C39.1, C58.1, C83.1, FB5.2
Other:
- moved on the sheet: C50, C51, FB1, FB2, R76, U4

Commit message: added production export
Parts:
- C1, C10, C2, C3, C35, C4, C5, C52, C6, C7, C8, C9: value 100n -> 100nF
- C20, C23, C25, C27, C29, C31, C33, C37, C39, C41, C43, C45, C69, C70, C73, C75, C80, C83, C85: value 0.1uF -> 100nF
- R10, R73, R74, R8: value 5.1k -> 2.7k
- R9: value 5.1k -> 1k
- U12: LCSC_Alt (none) -> C92004
- U4, U5: LCSC_Alt (none) -> C6186
Other:
- moved on the sheet: C1
Changed lines of the file:
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@@
 	)
 	(junction
-		(at 372.11 199.39)
+		(at 373.38 199.39)
 		(diameter 0)
 		(color 0 0 0 0)
@@
 	(wire
 		(pts
-			(xy 360.68 189.23) (xy 372.11 189.23)
+			(xy 360.68 189.23) (xy 373.38 189.23)
 		)
 		(stroke
@@
 	(wire
 		(pts
-			(xy 372.11 198.12) (xy 372.11 199.39)
+			(xy 373.38 198.12) (xy 373.38 199.39)
 		)
 		(stroke
@@
 	(wire
 		(pts
-			(xy 360.68 199.39) (xy 372.11 199.39)
+			(xy 360.68 199.39) (xy 375.92 199.39)
 		)
 		(stroke
@@
 	(wire
 		(pts
-			(xy 372.11 189.23) (xy 372.11 190.5)
+			(xy 373.38 189.23) (xy 373.38 190.5)
 		)
 		(stroke
@@
 	(wire
 		(pts
-			(xy 372.11 199.39) (xy 375.92 199.39)
-		)
-		(stroke
-			(width 0)
-			(type default)
-		)
-	)
-	(wire
-		(pts
 			(xy 217.17 224.79) (xy 217.17 215.9)
 		)
@@
 			)
 		)
-		(property "Value" "100n"
+		(property "Value" "100nF"
 			(at 368.3 218.4399 0)
 			(show_name no)
@@
 			)
 		)
-		(property "Value" "100n"
+		(property "Value" "100nF"
 			(at 364.49 195.5799 0)
 			(show_name no)
@@
 			)
 		)
-		(property "Value" "5.1k"
+		(property "Value" "2.7k"
 			(at 388.62 59.6899 0)
 			(show_name no)
@@
 			)
 		)
+		(property "LCSC_Alt" "C6186"
+			(at 185.42 62.23 0)
+			(hide yes)
+			(show_name no)
+			(do_not_autoplace no)
+			(effects
+				(font
+					(size 1.27 1.27)
+				)
+			)
+		)
 		(pin "1"
 		)
@@
 			)
 		)
-		(property "Value" "0.1uF"
+		(property "Value" "100nF"
 			(at 474.98 124.4599 0)
 			(show_name no)
@@
 			)
 		)
-		(property "Value" "0.1uF"
+		(property "Value" "100nF"
 			(at 474.98 143.5099 0)
 			(show_name no)
@@
 			)
 		)
-		(property "Value" "100n"
+		(property "Value" "100nF"
 			(at 328.93 218.4399 0)
 			(show_name no)
@@
 			)
 		)
-		(property "Value" "0.1uF"
+		(property "Value" "100nF"
 			(at 176.022 350.0119 0)
 			(show_name no)
@@
 			)
 		)
-		(property "Value" "0.1uF"
+		(property "Value" "100nF"
 			(at 525.78 143.5099 0)
 			(show_name no)
@@
 			)
 		)
-		(property "Value" "0.1uF"
+		(property "Value" "100nF"
 			(at 500.38 143.5099 0)
 			(show_name no)
@@
 			)
 		)
-		(property "Value" "0.1uF"
+		(property "Value" "100nF"
 			(at 474.98 88.8999 0)
 			(show_name no)
@@
 			)
 		)
-		(property "Value" "0.1uF"
+		(property "Value" "100nF"
 			(at 500.38 124.4599 0)
 			(show_name no)
@@
 			)
 		)
-		(property "Value" "100n"
+		(property "Value" "100nF"
 			(at 415.29 218.4399 0)
 			(show_name no)
@@
 			)
 		)
-		(property "Value" "0.1uF"
+		(property "Value" "100nF"
 			(at 474.98 105.4099 0)
 			(show_name no)
@@
 			)
 		)
-		(property "Value" "0.1uF"
+		(property "Value" "100nF"
 			(at 60.96 351.7899 0)
 			(show_name no)
@@
 			)
 		)
-		(property "Value" "0.1uF"
+		(property "Value" "100nF"
 			(at 500.38 72.3899 0)
 			(show_name no)
@@
 			)
 		)
-		(property "Value" "5.1k"
+		(property "Value" "1k"
 			(at 344.17 58.4199 0)
 			(show_name no)
@@
 			)
 		)
-		(property "Value" "0.1uF"
+		(property "Value" "100nF"
 			(at 472.44 53.3399 0)
 			(show_name no)
@@
 			)
 		)
-		(property "Value" "100n"
+		(property "Value" "100nF"
 			(at 427.99 218.4399 0)
 			(show_name no)
@@
 			)
 		)
-		(property "Value" "0.1uF"
+		(property "Value" "100nF"
 			(at 474.98 72.3899 0)
 			(show_name no)
@@
 			)
 		)
-		(property "Value" "0.1uF"
+		(property "Value" "100nF"
 			(at 500.38 88.8999 0)
 			(show_name no)
@@
 			)
 		)
-		(property "Value" "100n"
+		(property "Value" "100nF"
 			(at 378.46 218.4399 0)
 			(show_name no)
@@
 			)
 		)
+		(property "LCSC_Alt" "C6186"
+			(at 173.99 124.46 0)
+			(hide yes)
+			(show_name no)
+			(do_not_autoplace no)
+			(effects
+				(font
+					(size 1.27 1.27)
+				)
+			)
+		)
 		(pin "1"
 		)
@@
 			)
 		)
-		(property "Value" "100n"
+		(property "Value" "100nF"
 			(at 342.9 218.4399 0)
 			(show_name no)
@@
 			)
 		)
-		(property "Value" "100n"
+		(property "Value" "100nF"
 			(at 354.33 218.4399 0)
 			(show_name no)
@@
 			)
 		)
-		(property "Value" "0.1uF"
+		(property "Value" "100nF"
 			(at 497.84 53.3399 0)
 			(show_name no)
@@
 			)
 		)
-		(property "Value" "5.1k"
+		(property "Value" "2.7k"
 			(at 391.16 120.6499 0)
 			(show_name no)
@@
 			)
 		)
-		(property "Value" "5.1k"
+		(property "Value" "2.7k"
 			(at 330.2 58.4199 0)
 			(show_name no)
@@
 	(symbol
 		(lib_id "Device:C")
-		(at 372.11 194.31 0)
+		(at 373.38 194.31 0)
 		(unit 1)
 		(body_style 1)
@@
 		(fields_autoplaced yes)
 		(property "Reference" "C1"
-			(at 375.92 193.0399 0)
+			(at 377.19 193.0399 0)
 			(show_name no)
 			(do_not_autoplace no)
@@
 			)
 		)
-		(property "Value" "100n"
-			(at 375.92 195.5799 0)
+		(property "Value" "100nF"
+			(at 377.19 195.5799 0)
 			(show_name no)
 			(do_not_autoplace no)
@@
 		)
 		(property "Footprint" "Capacitor_SMD:C_0402_1005Metric_Pad0.74x0.62mm_HandSolder"
-			(at 373.0752 198.12 0)
+			(at 374.3452 198.12 0)
 			(hide yes)
 			(show_name no)
@@
 		)
 		(property "Datasheet" ""
-			(at 372.11 194.31 0)
+			(at 373.38 194.31 0)
 			(hide yes)
 			(show_name no)
@@
 		)
 		(property "Description" "Unpolarized capacitor"
-			(at 372.11 194.31 0)
+			(at 373.38 194.31 0)
 			(hide yes)
 			(show_name no)
@@
 			)
 		)
-		(property "Value" "0.1uF"
+		(property "Value" "100nF"
 			(at 183.388 393.7 0)
 			(show_name no)
@@
 			)
 		)
-		(property "Value" "0.1uF"
+		(property "Value" "100nF"
 			(at 124.46 355.5999 0)
 			(show_name no)
@@
 			)
 		)
-		(property "Value" "0.1uF"
+		(property "Value" "100nF"
 			(at 525.78 124.4599 0)
 			(show_name no)
@@
 			)
 		)
-		(property "Value" "0.1uF"
+		(property "Value" "100nF"
 			(at 228.6 205.7399 0)
 			(show_name no)
@@
 			)
 		)
-		(property "Value" "100n"
+		(property "Value" "100nF"
 			(at 403.86 218.4399 0)
 			(show_name no)
@@
 			)
 		)
-		(property "Value" "5.1k"
+		(property "Value" "2.7k"
 			(at 363.22 120.6499 0)
 			(show_name no)
@@
 			)
 		)
-		(property "Value" "0.1uF"
+		(property "Value" "100nF"
 			(at 251.46 205.7399 0)
 			(show_name no)
@@
 			)
 		)
-		(property "Value" "100n"
+		(property "Value" "100nF"
 			(at 392.43 218.4399 0)
 			(show_name no)
@@
 			)
 		)
-		(property "Value" "100n"
+		(property "Value" "100nF"
 			(at 350.52 195.5799 0)
 			(show_name no)
@@
 			(hide yes)
 			(show_name no)
+			(do_not_autoplace no)
+			(effects
+				(font
+					(size 1.27 1.27)
+				)
+			)
+		)
+		(property "LCSC_Alt" "C92004"
+			(at 67.31 394.97 0)
+			(hide yes)
+			(show_name no)
